Commit message: Editted:ImprovedCasterBallSlip

File: bot_bringup/urdf/bot_one.urdf (robot description, URDF)
Before this commit: robot Jeevan, 7 links, 6 joints
Joints:
- joint caster_joint: axis 0 0 1 -> (none); type continuous -> fixed

Commit message: Editted:CodeRefactored

File: bot_bringup/urdf/bot_one.urdf (robot description, URDF)
Before this commit: robot Jeevan, 7 links, 6 joints
Joints:
- joint laser_joint: axis 0 0 1 -> (none)

Commit message: Editted:CorrectedBaseLinkToWheels

File: bot_bringup/urdf/bot_one.urdf (robot description, URDF)
Before this commit: robot Jeevan, 7 links, 6 joints
Joints:
- joint wheel_left_joint: parent base_footprint -> base_link
- joint wheel_right_joint: parent base_footprint -> base_link
